File: BreadBoardPowerSupply.kicad_pcb (KiCad board)
At the start: 2 copper layers, 55 x 36 mm, 17 parts, among them J1 Barrel_Jack, J2 Conn_02x04_Odd_Even, J3 Conn_01x02_Pin, J4 Conn_01x02_Pin, J5 Conn_01x02_Pin, J6 Conn_01x02_Pin, U1 Mini Digital Voltometer, U2 LM317_TO-220, U3 Bread Board

Commit message: Update schematic and pcb
Parts:
- removed J3, J4, J5, J6: Conn_01x02_Pin, Connector_PinHeader_2.54mm:PinHeader_1x02_P2.54mm_Vertical
- removed U3: Bread Board, MyFootPrints:Breadboard
- added H1: MountingHole, MountingHole:MountingHole_2.2mm_M2, F.Cu at (115.3, 83.0)
- added H2: MountingHole, MountingHole:MountingHole_2.2mm_M2, F.Cu at (164.8, 83.0)
- added H3: MountingHole, MountingHole:MountingHole_2.2mm_M2, F.Cu at (115.3, 113.0)
- added H4: MountingHole, MountingHole:MountingHole_2.2mm_M2, F.Cu at (164.8, 113.0)
- moved C3 30.0 mm to (158.0, 113.0), turned to 90 degrees
- moved J2 24.5 mm to (163.4, 106.5), turned to 180 degrees
- moved R1 17.0 mm to (155.6, 98.4), turned to 180 degrees
- moved D1 15.7 mm to (140.7, 90.8)
- moved D2 9.38 mm to (144.0, 94.9), turned to 180 degrees
- moved S1 7.38 mm to (133.8, 91.0)
- moved C1 7.37 mm to (131.0, 83.7), turned to 90 degrees
- moved J1 4.87 mm to (123.9, 87.4)
- moved R2 4.54 mm to (141.4, 87.5)
- moved RV1 3.88 mm to (158.2, 93.5)
- moved U2 2.70 mm to (134.9, 84.1)
- moved U1 0.10 mm to (140.1, 104.7)
Routing:
- net /DC_OUT: track 0.00 -> 75.6 mm
- net /DC_IN: track 0.00 -> 45.2 mm
- net Net-(U2-ADJ): track 0.00 -> 39.0 mm
- net +12V: track 0.00 -> 17.9 mm
- net Net-(D2-A): track 0.00 -> 8.88 mm
- net /ON/OFF GREEN LED: track 0.00 -> 7.48 mm
- net Net-(D1-A): track 0.00 -> 3.62 mm
- net GND: vias 0 -> 50
- added copper zone on B.Cu, net GND
- added copper zone on F.Cu, net GND
Other:
- board text added: "Breadboard Power Supply"
- board text added: "D2"
- board text added: "DC Input"
- board text added: "DC OUT"
- board text added: "GND"
- board text added: "Michał Głuszak"
- board text added: "POWER ON/OFF"
