File: DesktopPowerSupply.kicad_pcb (KiCad board)
At the start: 2 copper layers, 55 x 36 mm, 16 parts, among them J1 Barrel_Jack, J2 Conn_02x04_Odd_Even, U1 Mini Digital Voltometer, U2 LM317_TO-220

Commit message: Rename project, end project
Other:
- board text added: "Desktop Power Supply"
- board text removed: "Breadboard Power Supply"
Changed lines of the file:
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@@
+	)
+	(gr_rect
+		(start 112.525 85.5)
+		(end 117.85 110.45)
+		(stroke
+			(width 0.1)
+			(type default)
+		)
+		(fill no)
+		(layer "User.1")
 	)
 	(gr_rect
@@
 		)
 	)
-	(gr_text "Breadboard Power Supply"
-		(at 115 100.25 270)
+	(gr_text "Desktop Power Supply"
+		(at 115 97.97 270)
 		(layer "F.SilkS" knockout)
 		(effects
@@
 	)
 	(gr_text "Michał Głuszak\n"
-		(at 116.375 100.25 270)
+		(at 116.35 97.97 270)
 		(layer "F.SilkS" knockout)
 		(effects
